Commit message: Update reference frame and add launch option for RViz in touch.launch; rename links and joints in URDF for touch configuration

File: omni_description/urdf/omni.urdf (robot description, URDF)
Before this commit: robot phantom_omni, 7 links, 6 joints
Links:
- removed link base
- removed link lower_arm
- removed link stylus
- removed link tip
- removed link torso
- removed link upper_arm
- removed link wrist
- added link touch_base; visual mesh filename=package://omni_description/meshes/base.stl
- added link touch_lower_arm; visual mesh filename=package://omni_description/meshes/lower_arm.stl
- added link touch_stylus; visual mesh filename=package://omni_description/meshes/pen.stl
- added link touch_tip; visual mesh filename=package://omni_description/meshes/tip.stl
- added link touch_torso; visual mesh filename=package://omni_description/meshes/torso.stl
- added link touch_upper_arm; visual mesh filename=package://omni_description/meshes/upper_arm.stl
- added link touch_wrist; visual mesh filename=package://omni_description/meshes/wrist.stl
- added link world
Joints:
- added joint world_to_base: type fixed, parent world, child touch_base, origin xyz=0 0 0 rpy=0 0 0
- joint elbow: child lower_arm -> touch_lower_arm; parent upper_arm -> touch_upper_arm
- joint pitch: child tip -> touch_tip; parent wrist -> touch_wrist
- joint roll: child stylus -> touch_stylus; parent tip -> touch_tip
- joint shoulder: child upper_arm -> touch_upper_arm; parent torso -> touch_torso
- joint waist: child torso -> touch_torso; parent base -> touch_base
- joint yaw: child wrist -> touch_wrist; parent lower_arm -> touch_lower_arm

Commit message: Add touch_force link and joint to URDF for enhanced robot interaction

File: omni_description/urdf/omni.urdf (robot description, URDF)
Before this commit: robot phantom_omni, 8 links, 7 joints
Links:
- added link touch_force; visual box size=0.01 0.01 0.01
Joints:
- added joint touch_tip_to_touch_force: type fixed, parent touch_base, child touch_force, origin xyz=0 0.1 0.3 rpy=0 0 3.14159
