Commit message: Rename omni to touch

File: touch_description/urdf/touch.urdf (robot description, URDF)
Before this commit: robot phantom_omni, 9 links, 8 joints
Links:
- link touch_base: geometry visual mesh filename=package://touch_description/meshes/base.stl
- link touch_lower_arm: geometry visual mesh filename=package://touch_description/meshes/lower_arm.stl
- link touch_stylus: geometry visual mesh filename=package://touch_description/meshes/pen.stl
- link touch_tip: geometry visual mesh filename=package://touch_description/meshes/tip.stl
- link touch_torso: geometry visual mesh filename=package://touch_description/meshes/torso.stl
- link touch_upper_arm: geometry visual mesh filename=package://touch_description/meshes/upper_arm.stl
- link touch_wrist: geometry visual mesh filename=package://touch_description/meshes/wrist.stl
